File: espa-max/espa-max.kicad_sch (KiCad schematic)
At the start: 38 parts, among them J1 Conn_01x11_Pin, J2 R-RJ45R08P-B000, J4 R-RJ45R08P-B000, U1 ESP32-S3-MINI-1-N8, U2 ESD7104MUTAG, U3 AP63203WU

Commit message: Rearranging folder structure and first efforts towards supporting CT clamps
Parts:
- removed J2, J4: R-RJ45R08P-B000, RRJ45R08PB000, symbol R-RJ45R08P-B000:R-RJ45R08P-B000
- added J3: RJ45_LED_Shielded_x2, HCTL HC-RJ45-5JA-2-5:undefined_HC-RJ45-5JA-2-5, symbol Connector:RJ45_LED_Shielded_x2
Connections:
- net GND: now also J3.19, J3.7
- net RJ45-1: now also J3.1, J3.13
- net RJ45-2: now also J3.14, J3.2
- net RJ45-3: now also J3.15, J3.3
- net RJ45-4: now also J3.16, J3.4
- net RJ45-5: now also J3.17, J3.5
- net RJ45-6: now also J3.18, J3.6
- net RJ45-8: now also J3.20, J3.8
- no-connect marks 24 -> 33
Other:
- added sheet energy-monitoring (energy-monitoring.kicad_sch)

Commit message: Misc updates from a while back. Committing before I do an update to use smaller components.
Parts:
- removed BOOT1: BOOT, Button_Switch_SMD:SW_SPST_PTS810, symbol Switch:SW_MEC_5E
- removed F1: 30V 500mA, Fuse:Fuse_1812_4532Metric, symbol Device:Fuse
- removed H2: MountingHole, MountingHole:MountingHole_3.2mm_M3, symbol Mechanical:MountingHole
- removed J1: Conn_01x11_Pin, Connector_PinHeader_2.54mm:PinHeader_1x11_P2.54mm_Vertical, symbol Connector:Conn_01x11_Pin
- removed RESET1: RESET, Button_Switch_SMD:SW_SPST_PTS810, symbol Switch:SW_MEC_5E
- removed U1: ESP32-S3-MINI-1-N8, ESP32-S3-MINI-1-N8:XCVR_ESP32-S3-MINI-1-N8, symbol ESP32-S3-MINI-1-N8:ESP32-S3-MINI-1-N8
- added C4: 10μF, Capacitor_SMD:C_0603_1608Metric, symbol Device:C
- added F2: 33V 500mA, PCM_Fuse_AKL:Fuse_1206_3216Metric, symbol Device:Fuse
- added J1: Screw_Terminal_01x10, TerminalBlock_Phoenix:TerminalBlock_Phoenix_MPT-0,5-10-2.54_1x10_P2.54mm_Horizontal, symbol Connector:Screw_Terminal_01x10
- added R11, R12: 10kΩ, Resistor_SMD:R_0603_1608Metric, symbol Device:R_Small
- added R13, R14, R15, R16: 330Ω, Resistor_SMD:R_0603_1608Metric, symbol Device:R
- added S1: BOOT, ALPS SKRPACE010:SW_SKRPACE010, symbol SKRPACE010:SKRPACE010
- added S2: RESET, ALPS SKRPACE010:SW_SKRPACE010, symbol SKRPACE010:SKRPACE010
- added U1: KH-PJ-328-SMT, 3.5mm-connector:AUDIO-SMD_KH-PJ-328-SMT, symbol 3.5mm-connector:KH-PJ-328-SMT
- added U5: ESP32-S3-MINI-1U, RF_Module:ESP32-S2-MINI-1U, symbol RF_Module:ESP32-S3-MINI-1U
Connections:
- net +12V_fused: now also F2.2
- net +3.3V: now also J1.1 (Pin_1), R11.2, U5.3 (3V3)
- net ESP32_EN: now also S2.3, S2.4, U5.45 (EN)
- net GND: now also J3.11, J3.21, J3.23, J3.9, C4.2, J1.10 (Pin_10), R12.1, S1.1, S1.2, S2.1, S2.2, U5.1 (GND), U5.2 (GND), U5.42 (GND), U5.43 (GND), U5.46 (GND), U5.47 (GND), U5.48 (GND), U5.49 (GND), U5.50 (GND), U5.51 (GND), U5.52 (GND), U5.53 (GND), U5.54 (GND), U5.55 (GND), U5.56 (GND), U5.57 (GND), U5.58 (GND), U5.59 (GND), U5.60 (GND), U5.61 (GND), U5.62 (GND), U5.63 (GND), U5.64 (GND), U5.65 (GND)
- net GPIO0: now also S1.3, S1.4, U5.4 (IO0)
- net GPIO1: now also J1.2 (Pin_2), U5.5 (IO1)
- net GPIO10: now also U1.3, U5.14 (IO10)
- net GPIO11: now also U5.15 (IO11)
- net GPIO12: now also U5.16 (IO12)
- net GPIO13: now also U5.17 (IO13)
- net GPIO14: now also U5.18 (IO14)
- net GPIO15: now also U5.19 (IO15)
- net GPIO16: now also U5.20 (IO16)
- net GPIO2: now also J1.3 (Pin_3), U5.6 (IO2)
- net GPIO21: now also U5.25 (IO21)
- net GPIO26: now also U5.26 (IO26)
- net GPIO3: now also J1.4 (Pin_4), U5.7 (IO3)
- net GPIO33: now also U5.28 (IO33)
- net GPIO34: now also U5.29 (IO34)
- net GPIO35: now also R13.1, U5.31 (IO35)
- net GPIO36: now also R16.1, U5.32 (IO36)
- net GPIO37: now also R14.1, U5.33 (IO37)
- net GPIO38: now also R15.1, U5.34 (IO38)
- net GPIO39: now also U5.35 (IO39)
- net GPIO4: now also J1.5 (Pin_5), U5.8 (IO4)
- net GPIO40: now also U1.5, U5.36 (IO40)
- net GPIO41: now also U5.37 (IO41)
- net GPIO42: now also U5.38 (IO42)
- net GPIO43: now also U5.39 (TXD0)
- net GPIO44: now also U5.40 (RXD0)
- net GPIO45: now also U5.41 (IO45)
- net GPIO46: now also U5.44 (IO46)
- net GPIO47: now also U5.27 (IO47)
- net GPIO48: now also U5.30 (IO48)
- net GPIO5: now also J1.6 (Pin_6), U5.9 (IO5)
- net GPIO6: now also J1.7 (Pin_7), U5.10 (IO6)
- net GPIO7: now also J1.8 (Pin_8), U5.11 (IO7)
- net GPIO8: now also J1.9 (Pin_9), U5.12 (IO8)
- net GPIO9: now also U5.13 (IO9)
- net I2C_SCL: now also U5.21 (IO17)
- net I2C_SDA: now also U5.22 (IO18)
- net USB_N: now also U5.23 (IO19)
- net USB_P: now also U5.24 (IO20)
- net at J3.22: now also R13.2
- net at J3.24: now also R14.2
- net at J3.10: now also R15.2
- net at J3.12: now also R16.2
- net RJ45-8 renamed +12V
- net +12V: now also F2.1
- new net: C4.1, R11.1, R12.2, U1.6
- no-connect marks 33 -> 23
Other:
- removed sheet energy-monitoring
- note added: "CT Clamp Connector"
- note added: "RJ-45 Connectors"
- note removed: "RJ-45 Connector"
- note removed: "RJ-45 Connector (Loop)"
- moved on the sheet: C5, C6, C7, C9, D1, D3, H1, H3, H4, J3A, J3B, L1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
