File: espa-mini/espa-mini.kicad_sch (KiCad schematic)
At the start: 35 parts, among them J1 Conn_01x11_Pin, J4 R-RJ45R08P-B000, U1 ESP32-S3-MINI-1-N8, U2 ESD7104MUTAG, U3 AP63203WU

Commit message: Misc updates from a while back. Committing before I do an update to use smaller components.
Parts:
- removed F1: 30V 500mA, Fuse:Fuse_1812_4532Metric, symbol Device:Fuse
- added F2: 33V 500mA, PCM_Fuse_AKL:Fuse_1206_3216Metric, symbol Device:Fuse
Connections:
- net +12V: now also F2.1
- net +12V_fused: now also F2.2

Commit message: Prepping for open source
Parts:
- C3: footprint Capacitor_SMD:C_0603_1608Metric -> Capacitor_SMD:C_0402_1005Metric; JLC Part# C15849 -> C52923
- R1, R2, R4: footprint Resistor_SMD:R_0603_1608Metric -> Resistor_SMD:R_0402_1005Metric; JLC Part# C23186 -> C25905
- R10, R9: footprint Resistor_SMD:R_0603_1608Metric -> Resistor_SMD:R_0402_1005Metric; JLC Part# C23138 -> C25104
- R3: footprint Resistor_SMD:R_0603_1608Metric -> Resistor_SMD:R_0402_1005Metric; JLC Part# C25804 -> C25744
- R5, R6, R7, R8: footprint Resistor_SMD:R_0603_1608Metric -> Resistor_SMD:R_0402_1005Metric
Connections:
- net SPA_RX: now reaches J4.5, R10.1
- net SPA_TX: now reaches J4.6, R9.1
- net SW: now reaches C6.1, L1.1, U3.5 (SW)
- net +12V_fused renamed VIN
Changed lines of the file:
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@@
 		)
 	)
-	(label "+12V_fused"
+	(label "VIN"
 		(at 40.64 143.51 0)
 		(effects
@@
 		)
 	)
+	(label "SPA_RX"
+		(at 245.11 140.97 0)
+		(effects
+			(font
+				(size 1.27 1.27)
+			)
+			(justify left bottom)
+		)
+	)
+	(label "SW"
+		(at 72.39 148.59 0)
+		(effects
+			(font
+				(size 1.27 1.27)
+			)
+			(justify left bottom)
+		)
+	)
+	(label "SPA_TX"
+		(at 209.55 140.97 180)
+		(effects
+			(font
+				(size 1.27 1.27)
+			)
+			(justify right bottom)
+		)
+	)
 	(label "GPIO5"
 		(at 143.51 62.23 0)
@@
 			)
 		)
-		(property "Footprint" "Resistor_SMD:R_0603_1608Metric"
+		(property "Footprint" "Resistor_SMD:R_0402_1005Metric"
 			(at 177.292 137.16 90)
 			(effects
@@
 			)
 		)
-		(property "Datasheet" "https://jlcpcb.com/partdetail/C22962"
+		(property "Datasheet" "https://jlcpcb.com/partdetail/C25091"
 			(at 179.07 137.16 0)
 			(effects
@@
 			)
 		)
-		(property "Footprint" "Resistor_SMD:R_0603_1608Metric"
+		(property "Footprint" "Resistor_SMD:R_0402_1005Metric"
 			(at 58.42 38.1 0)
 			(effects
@@
 			)
 		)
-		(property "Datasheet" "https://jlcpcb.com/partdetail/C23186"
+		(property "Datasheet" "https://jlcpcb.com/partdetail/C25905"
 			(at 58.42 38.1 0)
 			(effects
@@
 			)
 		)
-		(property "JLC Part#" "C23186"
+		(property "JLC Part#" "C25905"
 			(at 58.42 38.1 90)
 			(effects
@@
 			)
 		)
-		(property "Footprint" "Resistor_SMD:R_0603_1608Metric"
+		(property "Footprint" "Resistor_SMD:R_0402_1005Metric"
 			(at 52.07 35.56 0)
 			(effects
@@
 			)
 		)
-		(property "Datasheet" "https://jlcpcb.com/partdetail/C23186"
+		(property "Datasheet" "https://jlcpcb.com/partdetail/26648-0402WGF5101TCE/C25905"
 			(at 52.07 35.56 0)
 			(effects
@@
 			)
 		)
-		(property "JLC Part#" "C23186"
+		(property "JLC Part#" "C25905"
 			(at 52.07 35.56 90)
 			(effects
@@
 			)
 		)
-		(property "Footprint" "Resistor_SMD:R_0603_1608Metric"
+		(property "Footprint" "Resistor_SMD:R_0402_1005Metric"
 			(at 130.81 27.94 0)
 			(effects
@@
 			)
 		)
-		(property "Datasheet" "https://jlcpcb.com/partdetail/C25804"
+		(property "Datasheet" "https://jlcpcb.com/partdetail/C25744"
 			(at 130.81 27.94 0)
 			(effects
@@
 			)
 		)
-		(property "JLC Part#" "C25804"
+		(property "JLC Part#" "C25744"
 			(at 130.81 27.94 0)
 			(effects
@@
 			)
 		)
-		(property "Footprint" "Capacitor_SMD:C_0603_1608Metric"
+		(property "Footprint" "Capacitor_SMD:C_0402_1005Metric"
 			(at 119.38 38.1 0)
 			(effects
@@
 			)
 		)
-		(property "Datasheet" "https://jlcpcb.com/partdetail/C15849"
+		(property "Datasheet" "https://jlcpcb.com/partdetail/C52923"
 			(at 119.38 38.1 0)
 			(effects
@@
 			)
 		)
-		(property "JLC Part#" "C15849"
+		(property "JLC Part#" "C52923"
 			(at 119.38 38.1 0)
 			(effects
@@
 			)
 		)
-		(property "Footprint" "Resistor_SMD:R_0603_1608Metric"
+		(property "Footprint" "Resistor_SMD:R_0402_1005Metric"
 			(at 136.652 137.16 90)
 			(effects
@@
 			)
 		)
-		(property "Datasheet" "https://jlcpcb.com/partdetail/C22962"
+		(property "Datasheet" "https://jlcpcb.com/partdetail/C25091"
 			(at 138.43 137.16 0)
 			(effects
@@
 			)
 		)
-		(property "Footprint" "Resistor_SMD:R_0603_1608Metric"
+		(property "Footprint" "Resistor_SMD:R_0402_1005Metric"
 			(at 204.47 144.272 90)
 			(effects
@@
 			)
 		)
-		(property "Datasheet" "https://jlcpcb.com/partdetail/23865-0603WAF3300T5E/C23138"
+		(property "Datasheet" "https://jlcpcb.com/partdetail/C25104"
 			(at 204.47 146.05 0)
 			(effects
@@
 			)
 		)
-		(property "JLC Part#" "C23138"
+		(property "JLC Part#" "C25104"
 			(at 204.47 146.05 90)
 			(effects
@@
 			)
 		)
-		(property "Footprint" "Resistor_SMD:R_0603_1608Metric"
+		(property "Footprint" "Resistor_SMD:R_0402_1005Metric"
 			(at 254 147.828 90)
 			(effects
@@
 			)
 		)
-		(property "Datasheet" "https://jlcpcb.com/partdetail/23865-0603WAF3300T5E/C23138"
+		(property "Datasheet" "https://jlcpcb.com/partdetail/C25104"
 			(at 254 146.05 0)
 			(effects
@@
 			)
 		)
-		(property "JLC Part#" "C23138"
+		(property "JLC Part#" "C25104"
 			(at 254 146.05 90)
 			(effects
@@
 			)
 		)
-		(property "Footprint" "Resistor_SMD:R_0603_1608Metric"
+		(property "Footprint" "Resistor_SMD:R_0402_1005Metric"
 			(at 151.892 137.16 90)
 			(effects
@@
 			)
 		)
-		(property "Datasheet" "https://jlcpcb.com/partdetail/C22962"
+		(property "Datasheet" "https://jlcpcb.com/partdetail/C25091"
 			(at 153.67 137.16 0)
 			(effects
@@
 			)
 		)
-		(property "Footprint" "Resistor_SMD:R_0603_1608Metric"
+		(property "Footprint" "Resistor_SMD:R_0402_1005Metric"
 			(at 109.982 160.02 90)
 			(effects
@@
 			)
 		)
-		(property "Datasheet" "https://jlcpcb.com/partdetail/C23186"
+		(property "Datasheet" "https://jlcpcb.com/partdetail/C25905"
 			(at 111.76 160.02 0)
 			(effects
@@
 			)
 		)
-		(property "JLC Part#" "C23186"
+		(property "JLC Part#" "C25905"
 			(at 111.76 160.02 0)
 			(effects
@@
 			)
 		)
-		(property "Footprint" "Resistor_SMD:R_0603_1608Metric"
+		(property "Footprint" "Resistor_SMD:R_0402_1005Metric"
 			(at 164.592 137.16 90)
 			(effects
@@
 			)
 		)
-		(property "Datasheet" "https://jlcpcb.com/partdetail/C22962"
+		(property "Datasheet" "https://jlcpcb.com/partdetail/C25091"
 			(at 166.37 137.16 0)
 			(effects
